File: CapacitanceSelector.sch (EAGLE design)
At the start: 1 part

Commit message: Moving forward with it
Parts:
- removed S1: (no value), SparkFun-Electromechanical:SWITCH-DPDTEG2211
- added BLACK, RED: BINDING_POST, SparkFun-Connectors:BINDING_POST
- added C1: 10p, SparkFun-Capacitors:0.1UF-50V-20%(PTH)KIT-EZ
- added C2: 22p, SparkFun-Capacitors:0.1UF-50V-20%(PTH)KIT-EZ
- added C3: 100p, SparkFun-Capacitors:0.1UF-50V-20%(PTH)KIT-EZ
- added C4: 1n, SparkFun-Capacitors:0.1UF-50V-20%(PTH)KIT-EZ
- added C5: 10n, SparkFun-Capacitors:0.1UF-50V-20%(PTH)KIT-EZ
- added C6: 100n, SparkFun-Capacitors:0.1UF-50V-20%(PTH)KIT-EZ
- added DIAL1, DIAL2: 1x10, HokieGeek:SWITCH_ROTARY_1X12
- added LOGO1: OSHW-LOGOL, SparkFun-Aesthetics:OSHW-LOGOL
- added U$1: TOGGLE_SWITCH_DPDT_1, HokieGeek:TOGGLE_SWITCH_DPDT_1
Connections:
- new net N$1: DIAL1.COMMON, RED.P$1, U$1.3
- new net N$10: C6.2, DIAL1.7
- new net N$12: C1.2, C2.2, C3.2, C4.1, C5.1, C6.1, U$1.1, U$1.6
- new net N$3: BLACK.P$1, U$1.5
- new net N$4: DIAL2.COMMON, U$1.2
- new net N$5: C5.2, DIAL1.6
- new net N$6: C1.1, DIAL1.2
- new net N$7: C2.1, DIAL1.3
- new net N$8: C3.1, DIAL1.4
- new net N$9: C4.2, DIAL1.5
Changed lines of the file:
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@@
 <setting verticaltext="up"/>
 </settings>
-<grid distance="0.1" unitdist="inch" unit="inch" style="lines" multiple="1" display="no" altdistance="0.01" altunitdist="inch" altunit="inch"/>
+<grid distance="0.0125" unitdist="inch" unit="mm" style="lines" multiple="1" display="no" altdistance="0.00125" altunitdist="inch" altunit="mm"/>
 <layers>
 <layer number="1" name="Top" color="4" fill="1" visible="no" active="no"/>
@@
 <layer number="56" name="wert" color="7" fill="1" visible="no" active="no"/>
 <layer number="57" name="tCAD" color="7" fill="1" visible="no" active="no"/>
+<layer number="59" name="tCarbon" color="7" fill="1" visible="no" active="no"/>
+<layer number="60" name="bCarbon" color="7" fill="1" visible="no" active="no"/>
 <layer number="90" name="Modules" color="5" fill="1" visible="yes" active="yes"/>
 <layer number="91" name="Nets" color="2" fill="1" visible="yes" active="yes"/>
@@
 <layer number="112" name="tSilk" color="7" fill="1" visible="no" active="yes"/>
 <layer number="113" name="IDFDebug" color="4" fill="1" visible="no" active="yes"/>
+<layer number="114" name="Badge_Outline" color="7" fill="1" visible="yes" active="yes"/>
+<layer number="115" name="ReferenceISLANDS" color="7" fill="1" visible="yes" active="yes"/>
 <layer number="116" name="Patch_BOT" color="9" fill="4" visible="no" active="yes"/>
+<layer number="118" name="Rect_Pads" color="7" fill="1" visible="yes" active="yes"/>
 <layer number="121" name="_tsilk" color="7" fill="1" visible="no" active="yes"/>
 <layer number="122" name="_bsilk" color="7" fill="1" visible="no" active="yes"/>
@@
 <layer number="127" name="_tValues" color="7" fill="1" visible="no" active="yes"/>
 <layer number="128" name="_bValues" color="7" fill="1" visible="no" active="yes"/>
+<layer number="129" name="Mask" color="7" fill="1" visible="yes" active="yes"/>
 <layer number="131" name="tAdjust" color="7" fill="1" visible="no" active="yes"/>
 <layer number="132" name="bAdjust" color="7" fill="1" visible="no" active="yes"/>
@@
 <layer number="230" name="230bmp" color="7" fill="1" visible="yes" active="yes"/>
 <layer number="231" name="231bmp" color="7" fill="1" visible="yes" active="yes"/>
+<layer number="232" name="Eagle3D_PG2" color="7" fill="1" visible="no" active="no"/>
+<layer number="233" name="Eagle3D_PG3" color="7" fill="1" visible="no" active="no"/>
 <layer number="248" name="Housing" color="7" fill="1" visible="no" active="yes"/>
 <layer number="249" name="Edge" color="7" fill="1" visible="no" active="yes"/>
@@
 <layer number="251" name="SMDround" color="12" fill="11" visible="no" active="no"/>
 <layer number="254" name="cooling" color="7" fill="1" visible="no" active="yes"/>
+<layer number="255" name="routoute" color="7" fill="1" visible="yes" active="yes"/>
 </layers>
 <schematic xreflabel="%F%N/%S.%C%R" xrefpart="/%S.%C%R">
@@
 </classes>
 <parts>
-<part name="S1" library="SparkFun-Electromechanical" deviceset="SWITCH-DPDT" device="EG2211"/>
+<part name="DIAL1" library="HokieGeek" deviceset="SWITCH_ROTARY_1X12" device="" value="1x10"/>
+<part name="DIAL2" library="HokieGeek" deviceset="SWITCH_ROTARY_1X12" device="" value="1x10"/>
+<part name="RED" library="SparkFun-Connectors" deviceset="BINDING_POST" device=""/>
+<part name="BLACK" library="SparkFun-Connectors" deviceset="BINDING_POST" device=""/>
+<part name="LOGO1" library="SparkFun-Aesthetics" deviceset="OSHW-LOGO" device="L"/>
+<part name="U$1" library="HokieGeek" deviceset="TOGGLE_SWITCH_DPDT_1" device=""/>
+<part name="C1" library="SparkFun-Capacitors" deviceset="0.1UF-50V-20%(PTH)" device="KIT-EZ" value="10p"/>
+<part name="C2" library="SparkFun-Capacitors" deviceset="0.1UF-50V-20%(PTH)" device="KIT-EZ" value="22p"/>
+<part name="C3" library="SparkFun-Capacitors" deviceset="0.1UF-50V-20%(PTH)" device="KIT-EZ" value="100p"/>
+<part name="C4" library="SparkFun-Capacitors" deviceset="0.1UF-50V-20%(PTH)" device="KIT-EZ" value="1n"/>
+<part name="C5" library="SparkFun-Capacitors" deviceset="0.1UF-50V-20%(PTH)" device="KIT-EZ" value="10n"/>
+<part name="C6" library="SparkFun-Capacitors" deviceset="0.1UF-50V-20%(PTH)" device="KIT-EZ" value="100n"/>
 </parts>
 <sheets>
@@
 </plain>
 <instances>
-<instance part="S1" gate="G$1" x="96.52" y="142.24"/>
+<instance part="DIAL1" gate="G$1" x="27.94" y="22.86" rot="R270"/>
+<instance part="DIAL2" gate="G$1" x="73.66" y="22.86" rot="R270"/>
+<instance part="RED" gate="G$1" x="15.24" y="55.88" rot="R180"/>
+<instance part="BLACK" gate="G$1" x="101.6" y="53.34"/>
+<instance part="LOGO1" gate="G$1" x="94.615" y="10.16"/>
+<instance part="U$1" gate="G$1" x="53.34" y="55.88" rot="R180"/>
+<instance part="C1" gate="G$1" x="45.72" y="27.94" rot="R90"/>
+<instance part="C2" gate="G$1" x="45.72" y="22.86" rot="R90"/>
+<instance part="C3" gate="G$1" x="45.72" y="17.78" rot="R90"/>
+<instance part="C4" gate="G$1" x="35.56" y="7.62" rot="R180"/>
+<instance part="C5" gate="G$1" x="30.48" y="7.62" rot="R180"/>
+<instance part="C6" gate="G$1" x="25.4" y="7.62" rot="R180"/>
 </instances>
 <busses>
 </busses>
 <nets>
+<net name="N$1" class="0">
+<segment>
+<pinref part="DIAL1" gate="G$1" pin="COMMON"/>
+<wire x1="27.94" y1="35.56" x2="27.94" y2="55.88" width="0.1524" layer="91"/>
+<pinref part="RED" gate="G$1" pin="P$1"/>
+<wire x1="27.94" y1="55.88" x2="17.78" y2="55.88" width="0.1524" layer="91"/>
+<wire x1="48.26" y1="55.88" x2="27.94" y2="55.88" width="0.1524" layer="91"/>
+<junction x="27.94" y="55.88"/>
+<pinref part="U$1" gate="G$1" pin="3"/>
+</segment>
+</net>
+<net name="N$3" class="0">
+<segment>
+<pinref part="BLACK" gate="G$1" pin="P$1"/>
+<wire x1="99.06" y1="53.34" x2="88.9" y2="53.34" width="0.1524" layer="91"/>
+<wire x1="88.9" y1="53.34" x2="88.9" y2="38.1" width="0.1524" layer="91"/>
+<junction x="88.9" y="53.34"/>
+<wire x1="58.42" y1="60.96" x2="88.9" y2="60.96" width="0.1524" layer="91"/>
+<wire x1="88.9" y1="60.96" x2="88.9" y2="53.34" width="0.1524" layer="91"/>
+<pinref part="U$1" gate="G$1" pin="5"/>
+</segment>
+</net>
+<net name="N$4" class="0">
+<segment>
+<pinref part="DIAL2" gate="G$1" pin="COMMON"/>
+<wire x1="73.66" y1="35.56" x2="73.66" y2="53.34" width="0.1524" layer="91"/>
+<wire x1="73.66" y1="53.34" x2="58.42" y2="53.34" width="0.1524" layer="91"/>
+<pinref part="U$1" gate="G$1" pin="2"/>
+</segment>
+</net>
+<net name="N$6" class="0">
+<segment>
+<pinref part="DIAL1" gate="G$1" pin="2"/>
+<pinref part="C1" gate="G$1" pin="1"/>
+</segment>
+</net>
+<net name="N$7" class="0">
+<segment>
+<pinref part="DIAL1" gate="G$1" pin="3"/>
+<pinref part="C2" gate="G$1" pin="1"/>
+</segment>
+</net>
+<net name="N$8" class="0">
+<segment>
+<pinref part="DIAL1" gate="G$1" pin="4"/>
+<pinref part="C3" gate="G$1" pin="1"/>
+</segment>
+</net>
+<net name="N$9" class="0">
+<segment>
+<pinref part="DIAL1" gate="G$1" pin="5"/>
+<pinref part="C4" gate="G$1" pin="2"/>
+</segment>
+</net>
+<net name="N$5" class="0">
+<segment>
+<pinref part="DIAL1" gate="G$1" pin="6"/>
+<pinref part="C5" gate="G$1" pin="2"/>
+</segment>
+</net>
+<net name="N$10" class="0">
+<segment>
+<pinref part="DIAL1" gate="G$1" pin="7"/>
+<pinref part="C6" gate="G$1" pin="2"/>
+</segment>
+</net>
+<net name="N$12" class="0">
+<segment>
+<wire x1="48.26" y1="22.86" x2="50.165" y2="22.86" width="0.1524" layer="91"/>
+<pinref part="C2" gate="G$1" pin="2"/>
+<pinref part="C6" gate="G$1" pin="1"/>
+<wire x1="25.4" y1="2.54" x2="25.4" y2="0.3175" width="0.1524" layer="91"/>
+<pinref part="C3" gate="G$1" pin="2"/>
+<wire x1="48.26" y1="17.78" x2="50.165" y2="17.78" width="0.1524" layer="91"/>
+<wire x1="25.4" y1="0.3175" x2="30.48" y2="0.3175" width="0.1524" layer="91"/>
+<wire x1="30.48" y1="0.3175" x2="35.56" y2="0.3175" width="0.1524" layer="91"/>
+<wire x1="35.56" y1="0.3175" x2="50.165" y2="0.3175" width="0.1524" layer="91"/>
+<wire x1="50.165" y1="0.3175" x2="50.165" y2="17.78" width="0.1524" layer="91"/>
+<wire x1="50.165" y1="17.78" x2="50.165" y2="22.86" width="0.1524" layer="91"/>
+<pinref part="C1" gate="G$1" pin="2"/>
+<wire x1="50.165" y1="22.86" x2="50.165" y2="27.94" width="0.1524" layer="91"/>
+<wire x1="48.26" y1="27.94" x2="50.165" y2="27.94" width="0.1524" layer="91"/>
+<wire x1="50.165" y1="27.94" x2="50.165" y2="40.64" width="0.1524" layer="91"/>
+<wire x1="50.165" y1="40.64" x2="43.18" y2="40.64" width="0.1524" layer="91"/>
+<junction x="25.4" y="0.3175"/>
+<junction x="50.165" y="27.94"/>
+<junction x="50.165" y="22.86"/>
+<junction x="50.165" y="17.78"/>
+<wire x1="48.26" y1="63.5" x2="43.18" y2="63.5" width="0.1524" layer="91"/>
+<wire x1="43.18" y1="63.5" x2="43.18" y2="50.8" width="0.1524" layer="91"/>
+<wire x1="48.26" y1="50.8" x2="43.18" y2="50.8" width="0.1524" layer="91"/>
+<pinref part="U$1" gate="G$1" pin="1"/>
+<pinref part="U$1" gate="G$1" pin="6"/>
+<wire x1="43.18" y1="40.64" x2="43.18" y2="50.8" width="0.1524" layer="91"/>
+<junction x="43.18" y="50.8"/>
+<pinref part="C5" gate="G$1" pin="1"/>
+<wire x1="30.48" y1="2.54" x2="30.48" y2="0.3175" width="0.1524" layer="91"/>
+<junction x="30.48" y="0.3175"/>
+<pinref part="C4" gate="G$1" pin="1"/>
+<wire x1="35.56" y1="2.54" x2="35.56" y2="0.3175" width="0.1524" layer="91"/>
+<junction x="35.56" y="0.3175"/>
+</segment>
+</net>
 </nets>
 </sheet>
